Commit message: 24-10-18

File: cra_description/urdf/cr3_robot.xacro.urdf (robot description, URDF)
Before this commit: robot cr3_robot, 9 links, 8 joints
Links:
- added link gripper_dh; collision mesh filename=file://$(find cra_description)/meshes/cr3/gripper_dh.STL; visual mesh filename=file://$(find cra_description)/meshes/cr3/gripper_dh.STL
Joints:
- added joint joint_gripper_dh: type fixed, parent Link6, child gripper_dh, origin xyz=0 0 0.1065 rpy=0 0 0, axis 0 0 1

File: cra_moveit_config/config/gazebo_cr3_robot.urdf (robot description, URDF)
Before this commit: robot cr3_robot, 9 links, 8 joints
Links:
- added link gripper_dh, mass 0.1; collision mesh filename=file:///home/ubuntu/eyeAhand/src/cra_description/meshes/cr3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; visual mesh filename=file:///home/ubuntu/eyeAhand/src/cra_description/meshes/cr3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
- link Link1: geometry collision mesh filename=file:///home/ubuntu/eyeAhand/src/cra_description/meshes/cr3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; visual mesh filename=file:///home/ubuntu/eyeAhand/src/cra_description/meshes/cr3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
- link Link2: geometry collision mesh filename=file:///home/ubuntu/eyeAhand/src/cra_description/meshes/cr3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; visual mesh filename=file:///home/ubuntu/eyeAhand/src/cra_description/meshes/cr3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
- link Link3: geometry collision mesh filename=file:///home/ubuntu/eyeAhand/src/cra_description/meshes/cr3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; visual mesh filename=file:///home/ubuntu/eyeAhand/src/cra_description/meshes/cr3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
- link Link4: geometry collision mesh filename=file:///home/ubuntu/eyeAhand/src/cra_description/meshes/cr3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; visual mesh filename=file:///home/ubuntu/eyeAhand/src/cra_description/meshes/cr3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
- link Link5: geometry collision mesh filename=file:///home/ubuntu/eyeAhand/src/cra_description/meshes/cr3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; visual mesh filename=file:///home/ubuntu/eyeAhand/src/cra_description/meshes/cr3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
- link Link6: geometry collision mesh filename=file:///home/ubuntu/eyeAhand/src/cra_description/meshes/cr3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; visual mesh filename=file:///home/ubuntu/eyeAhand/src/cra_description/meshes/cr3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
- link base_link: geometry collision mesh filename=file:///home/ubuntu/eyeAhand/src/cra_description/meshes/cr3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; visual mesh filename=file:///home/ubuntu/eyeAhand/src/cra_description/meshes/cr3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
Joints:
- added joint joint_gripper_dh: type fixed, parent Link6, child gripper_dh, origin xyz=0 0 0 rpy=0 0 0, axis 0 0 1

Commit message: test

File: cra_description/urdf/cr3_robot.xacro.urdf (robot description, URDF)
Before this commit: robot cr3_robot, 10 links, 9 joints
Joints:
- joint joint_gripper_dh: origin xyz=0 0 0.1065 rpy=0 0 0 -> xyz=0 0 0.1695 rpy=0 0 0
